File: eagle/SparkySpecialK.sch (EAGLE design)
At the start: 23 parts, among them CN1 MiniB USB, IC1 ATMEGA32U4-AU, X3 16MHz

Commit message: updated connections
Connections:
- net A0 renamed A0/DOWN
- net A1 renamed A1/LEFT
- net A2 renamed A2/HOME
- net A3 renamed A3/1P
- net A4 renamed A4/3P
- net D10 renamed D10/SELECT
- net D12 renamed D12/1K
- net D13 renamed D13/UP
- net D2 renamed D2/4K
- net D3 renamed D3/2K
- net D4 renamed D4/3K
- net D5 renamed D5/RIGHT
- net D6 renamed D6/4P
- net D7 renamed D7/DATA_OUT
- net D8 renamed D8/2P
- net D9 renamed D9/START
Changed lines of the file:
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@@
 </segment>
 </net>
-<net name="D3" class="0">
+<net name="D3/2K" class="0">
 <segment>
 <wire x1="154.94" y1="-142.24" x2="177.8" y2="-142.24" width="0.1524" layer="91"/>
@@
 </segment>
 </net>
-<net name="D2" class="0">
+<net name="D2/4K" class="0">
 <segment>
 <wire x1="154.94" y1="-139.7" x2="177.8" y2="-139.7" width="0.1524" layer="91"/>
@@
 </segment>
 </net>
-<net name="D6" class="0">
+<net name="D6/4P" class="0">
 <segment>
 <wire x1="154.94" y1="-124.46" x2="177.8" y2="-124.46" width="0.1524" layer="91"/>
@@
 </segment>
 </net>
-<net name="D8" class="0">
+<net name="D8/2P" class="0">
 <segment>
 <wire x1="154.94" y1="-109.22" x2="177.8" y2="-109.22" width="0.1524" layer="91"/>
@@
 </segment>
 </net>
-<net name="D12" class="0">
+<net name="D12/1K" class="0">
 <segment>
 <wire x1="154.94" y1="-127" x2="177.8" y2="-127" width="0.1524" layer="91"/>
@@
 </segment>
 </net>
-<net name="D4" class="0">
+<net name="D4/3K" class="0">
 <segment>
 <wire x1="154.94" y1="-132.08" x2="177.8" y2="-132.08" width="0.1524" layer="91"/>
@@
 </segment>
 </net>
-<net name="A4" class="0">
+<net name="A4/3P" class="0">
 <segment>
 <wire x1="154.94" y1="-71.12" x2="177.8" y2="-71.12" width="0.1524" layer="91"/>
@@
 </segment>
 </net>
-<net name="A3" class="0">
+<net name="A3/1P" class="0">
 <segment>
 <wire x1="154.94" y1="-73.66" x2="177.8" y2="-73.66" width="0.1524" layer="91"/>
@@
 </segment>
 </net>
-<net name="A2" class="0">
+<net name="A2/HOME" class="0">
 <segment>
 <wire x1="154.94" y1="-76.2" x2="177.8" y2="-76.2" width="0.1524" layer="91"/>
@@
 </segment>
 </net>
-<net name="A1" class="0">
-<segment>
-<wire x1="154.94" y1="-78.74" x2="177.8" y2="-78.74" width="0.1524" layer="91"/>
-<label x="180.34" y="-78.74" size="1.778" layer="95"/>
-<pinref part="IC1" gate="G$1" pin="PF6(ADC6/TDO)"/>
-</segment>
-<segment>
-<pinref part="U$1" gate="G$1" pin="4"/>
-<wire x1="144.78" y1="-5.08" x2="152.4" y2="-5.08" width="0.1524" layer="91"/>
-<label x="154.94" y="-5.08" size="1.778" layer="95"/>
-</segment>
-</net>
-<net name="A0" class="0">
+<net name="A0/DOWN" class="0">
 <segment>
 <wire x1="154.94" y1="-81.28" x2="177.8" y2="-81.28" width="0.1524" layer="91"/>
@@
 </segment>
 </net>
-<net name="D7" class="0">
+<net name="D7/DATA_OUT" class="0">
 <segment>
 <wire x1="154.94" y1="-88.9" x2="177.8" y2="-88.9" width="0.1524" layer="91"/>
@@
 </segment>
 </net>
-<net name="D5" class="0">
+<net name="D5/RIGHT" class="0">
 <segment>
 <wire x1="154.94" y1="-93.98" x2="177.8" y2="-93.98" width="0.1524" layer="91"/>
@@
 </segment>
 </net>
-<net name="D13" class="0">
+<net name="D13/UP" class="0">
 <segment>
 <wire x1="154.94" y1="-96.52" x2="177.8" y2="-96.52" width="0.1524" layer="91"/>
@@
 </segment>
 </net>
-<net name="D10" class="0">
+<net name="D10/SELECT" class="0">
 <segment>
 <wire x1="154.94" y1="-104.14" x2="177.8" y2="-104.14" width="0.1524" layer="91"/>
@@
 </segment>
 </net>
-<net name="D9" class="0">
+<net name="D9/START" class="0">
 <segment>
 <wire x1="154.94" y1="-106.68" x2="177.8" y2="-106.68" width="0.1524" layer="91"/>
@@
 </segment>
 </net>
+<net name="A1/LEFT" class="0">
+<segment>
+<pinref part="U$1" gate="G$1" pin="4"/>
+<wire x1="144.78" y1="-5.08" x2="152.4" y2="-5.08" width="0.1524" layer="91"/>
+<label x="154.94" y="-5.08" size="1.778" layer="95"/>
+</segment>
+<segment>
+<wire x1="154.94" y1="-78.74" x2="177.8" y2="-78.74" width="0.1524" layer="91"/>
+<label x="180.34" y="-78.74" size="1.778" layer="95"/>
+<pinref part="IC1" gate="G$1" pin="PF6(ADC6/TDO)"/>
+</segment>
+</net>
